File: OpenFlowMeter.kicad_pcb (KiCad board)
At the start: 2 copper layers, 74.5 x 28 mm, 109 parts, among them J1 Screw_Terminal_01x02, J2 Screw_Terminal_01x02, J3 Conn_01x06, J4 Conn_02x03_Odd_Even, J5 Conn_01x03, J6 Conn_02x04_Odd_Even, J7 Conn_02x03_Odd_Even, Q1 BC856, Q2 BC856, U1 LT1492, U2 STM32F103C8Tx, U3 LT1492, U4 R-78C3.3-1.0, U5 SN65HVD231, U6 LT1492, U7 24LC64, Y1 12 MHz

Commit message: included values from simulation
added values to those components, which did not had one
Parts:
- C1, C2, C3, C4: value 100n -> 100n 50V
- C10: value C -> 1u 50V
- C11: value C -> 100n 50V
- C12, C14, C15, C16, C17, C18: value C -> 100n
- C13: value C -> 1u
- C19, C20: value C -> 27p
- C7, C8: value 100n -> 10n
- R17, R3: value 47k -> 100k
- R22, R29, R30, R8: value 1k -> 10k
Changed lines of the file:
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@@
       (effects (font (size 1 1) (thickness 0.15)))
     )
-    (fp_text value "47k" (at 0 1.43) (layer "F.Fab")
+    (fp_text value "100k" (at 0 1.43) (layer "F.Fab")
       (effects (font (size 1 1) (thickness 0.15)))
     )
@@
       (effects (font (size 1 1) (thickness 0.15)))
     )
-    (fp_text value "47k" (at 0 1.43) (layer "F.Fab")
+    (fp_text value "100k" (at 0 1.43) (layer "F.Fab")
       (effects (font (size 1 1) (thickness 0.15)))
     )
@@
       (effects (font (size 1 1) (thickness 0.15)))
     )
-    (fp_text value "100n" (at 0 1.43 -90) (layer "F.Fab")
+    (fp_text value "10n" (at 0 1.43 -90) (layer "F.Fab")
       (effects (font (size 1 1) (thickness 0.15)))
     )
@@
       (effects (font (size 1 1) (thickness 0.15)))
     )
-    (fp_text value "100n" (at 0 1.43 90) (layer "F.Fab")
+    (fp_text value "10n" (at 0 1.43 90) (layer "F.Fab")
       (effects (font (size 1 1) (thickness 0.15)))
     )
@@
       (effects (font (size 1 1) (thickness 0.15)))
     )
-    (fp_text value "1k" (at 0 1.43 90) (layer "F.Fab")
+    (fp_text value "10k" (at 0 1.43 90) (layer "F.Fab")
       (effects (font (size 1 1) (thickness 0.15)))
     )
@@
       (effects (font (size 1 1) (thickness 0.15)))
     )
-    (fp_text value "1k" (at 0 1.43 -90) (layer "F.Fab")
+    (fp_text value "10k" (at 0 1.43 -90) (layer "F.Fab")
       (effects (font (size 1 1) (thickness 0.15)))
     )
@@
       (effects (font (size 1 1) (thickness 0.15)))
     )
-    (fp_text value "1k" (at 0 1.43) (layer "F.Fab")
+    (fp_text value "10k" (at 0 1.43) (layer "F.Fab")
       (effects (font (size 1 1) (thickness 0.15)))
     )
@@
       (effects (font (size 1 1) (thickness 0.15)))
     )
-    (fp_text value "1k" (at 0 1.43) (layer "F.Fab")
+    (fp_text value "10k" (at 0 1.43) (layer "F.Fab")
       (effects (font (size 1 1) (thickness 0.15)))
     )
@@
       (effects (font (size 1 1) (thickness 0.15)))
     )
-    (fp_text value "C" (at 0 1.43 45) (layer "F.Fab")
+    (fp_text value "100n" (at 0 1.43 45) (layer "F.Fab")
       (effects (font (size 1 1) (thickness 0.15)))
     )
@@
       (effects (font (size 1 1) (thickness 0.15)))
     )
-    (fp_text value "C" (at 0 1.43 -135) (layer "F.Fab")
+    (fp_text value "27p" (at 0 1.43 -135) (layer "F.Fab")
       (effects (font (size 1 1) (thickness 0.15)))
     )
@@
       (effects (font (size 1 1) (thickness 0.15)))
     )
-    (fp_text value "C" (at 0 1.43) (layer "F.Fab")
+    (fp_text value "1u" (at 0 1.43) (layer "F.Fab")
       (effects (font (size 1 1) (thickness 0.15)))
     )
@@
       (effects (font (size 1 1) (thickness 0.15)))
     )
-    (fp_text value "C" (at 0 1.43 -135) (layer "F.Fab")
+    (fp_text value "100n" (at 0 1.43 -135) (layer "F.Fab")
       (effects (font (size 1 1) (thickness 0.15)))
     )
@@
       (effects (font (size 1 1) (thickness 0.15)))
     )
-    (fp_text value "C" (at 0 1.43 45) (layer "F.Fab")
+    (fp_text value "100n" (at 0 1.43 45) (layer "F.Fab")
       (effects (font (size 1 1) (thickness 0.15)))
     )
@@
       (effects (font (size 1 1) (thickness 0.15)))
     )
-    (fp_text value "C" (at 0 1.43 -45) (layer "F.Fab")
+    (fp_text value "100n" (at 0 1.43 -45) (layer "F.Fab")
       (effects (font (size 1 1) (thickness 0.15)))
     )
@@
       (effects (font (size 1 1) (thickness 0.15)))
     )
-    (fp_text value "C" (at 0 1.43 135) (layer "F.Fab")
+    (fp_text value "100n" (at 0 1.43 135) (layer "F.Fab")
       (effects (font (size 1 1) (thickness 0.15)))
     )
@@
       (effects (font (size 1 1) (thickness 0.15)))
     )
-    (fp_text value "C" (at 0 1.43) (layer "F.Fab")
+    (fp_text value "100n 50V" (at 0 1.43) (layer "F.Fab")
       (effects (font (size 1 1) (thickness 0.15)))
     )
@@
       (effects (font (size 1 1) (thickness 0.15)))
     )
-    (fp_text value "C" (at 0 1.43 -45) (layer "F.Fab")
+    (fp_text value "27p" (at 0 1.43 -45) (layer "F.Fab")
       (effects (font (size 1 1) (thickness 0.15)))
     )
@@
       (effects (font (size 1 1) (thickness 0.15)))
     )
-    (fp_text value "C" (at 0 1.43) (layer "F.Fab")
+    (fp_text value "100n" (at 0 1.43) (layer "F.Fab")
       (effects (font (size 1 1) (thickness 0.15)))
     )
@@
       (effects (font (size 1 1) (thickness 0.15)))
     )
-    (fp_text value "C" (at 0 1.43) (layer "F.Fab")
+    (fp_text value "1u 50V" (at 0 1.43) (layer "F.Fab")
       (effects (font (size 1 1) (thickness 0.15)))
     )
@@
       (effects (font (size 1 1) (thickness 0.15)) (justify mirror))
     )
-    (fp_text value "100n" (at 0 -1.43) (layer "B.Fab")
+    (fp_text value "100n 50V" (at 0 -1.43) (layer "B.Fab")
       (effects (font (size 1 1) (thickness 0.15)) (justify mirror))
     )
@@
       (effects (font (size 1 1) (thickness 0.15)) (justify mirror))
     )
-    (fp_text value "100n" (at 0 -1.43) (layer "B.Fab")
+    (fp_text value "100n 50V" (at 0 -1.43) (layer "B.Fab")
       (effects (font (size 1 1) (thickness 0.15)) (justify mirror))
     )
@@
       (effects (font (size 1 1) (thickness 0.15)) (justify mirror))
     )
-    (fp_text value "100n" (at 0 -1.43) (layer "B.Fab")
+    (fp_text value "100n 50V" (at 0 -1.43) (layer "B.Fab")
       (effects (font (size 1 1) (thickness 0.15)) (justify mirror))
     )
@@
       (effects (font (size 1 1) (thickness 0.15)) (justify mirror))
     )
-    (fp_text value "100n" (at 0 -1.43) (layer "B.Fab")
+    (fp_text value "100n 50V" (at 0 -1.43) (layer "B.Fab")
       (effects (font (size 1 1) (thickness 0.15)) (justify mirror))
     )
