File: OpenFlowMeter_PWM_Filter.kicad_sch (KiCad schematic)
At the start: 10 parts, among them U3 LT1492

Commit message: added company to all schematic pages
Other:
- company: (none) -> Jochen Steinmann
Changed lines of the file:
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@@
 (kicad_sch (version 20211123) (generator eeschema)
   (paper "A4")
+  (title_block
+    (rev "2")
+    (company "Jochen Steinmann")
+  )
   (junction (at 130.81 127) (diameter 0) (color 0 0 0 0)
   )
