File: OpenFlowMeter_I2Ccomponents.kicad_sch (KiCad schematic)
At the start: 10 parts, among them U10 BME680, U7 24LC64, U9 TMP100

Commit message: some tweak regarding BOM
Parts:
- JP2, JP3: now left out of the parts list
Changed lines of the file:
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@@
   )
   (symbol (lib_id "Jumper:Jumper_2_Bridged") (at 246.38 49.53 90) (unit 1)
-    (in_bom yes) (on_board yes) (dnp no) (fields_autoplaced)
+    (in_bom no) (on_board yes) (dnp no) (fields_autoplaced)
     (property "Reference" "JP2" (at 247.523 50.009 90)
       (effects (font (size 1.27 1.27)) (justify right))
@@
   )
   (symbol (lib_id "Jumper:SolderJumper_3_Bridged12") (at 257.81 142.24 270) (mirror x) (unit 1)
-    (in_bom yes) (on_board yes) (dnp no) (fields_autoplaced)
+    (in_bom no) (on_board yes) (dnp no) (fields_autoplaced)
     (property "Reference" "JP3" (at 260.35 142.2399 90)
       (effects (font (size 1.27 1.27)) (justify left))
