File: differential_ampl.kicad_sch (KiCad schematic)
At the start: 10 parts, among them U3 LT1492

Commit message: updated KiCAD version
Parts:
- renumbered C9 to C44, R8 to R54, R29 to R55, R29 to R56, R29 to R57, R29 to R68, R8 to R69, R8 to R70, R8 to R71, U3 to U13
